File: Hardware/L6-FBV3-Clone/L6-FBV3-Clone.sch (KiCad schematic (older format))
At the start: 25 parts, among them J1 Conn_02x20_Odd_Even, SW1 SW_Push, SW10 SW_Push, SW11 SW_Push, SW12 SW_Push, SW2 SW_Push, SW3 SW_Push, SW4 SW_Push, SW5 SW_Push, SW6 SW_Push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

Commit message: Updated schematic
Parts:
- D2: value TBD -> ALT
Connections:
- net TBD is gone; now on net ALT: SW12.1
- net BNK_DWN: now also J1.11 (Pin_11); no longer J1.16 (Pin_16)
- net BNK_UP: now also J1.7 (Pin_7); no longer J1.12 (Pin_12)
- net CLK: now also J1.38 (Pin_38)
- net DIN: now also J1.36 (Pin_36)
- net FX1: now also J1.13 (Pin_13); no longer J1.35 (Pin_35)
- net FX3: now also J1.29 (Pin_29); no longer J1.13 (Pin_13)
- net FX4: now also J1.31 (Pin_31); no longer J1.11 (Pin_11)
- net FX5: now also J1.33 (Pin_33); no longer J1.38 (Pin_38)
- net LOAD: now also J1.40 (Pin_40)
- net PRE_A: now also J1.35 (Pin_35)
- net PRE_B: now also J1.37 (Pin_37)
- net PRE_C: now also J1.12 (Pin_12)
- net PRE_D: now also J1.14 (Pin_14)
- net ALT: now reaches J1.18 (Pin_18)
Changed lines of the file:
@@
 P 10400 3250
 F 0 "D2" V 10439 3132 50  0000 R CNN
-F 1 "TBD" V 10348 3132 50  0000 R CNN
+F 1 "ALT" V 10348 3132 50  0000 R CNN
 F 2 "" H 10400 3250 50  0001 C CNN
 F 3 "~" H 10400 3250 50  0001 C CNN
@@
 BNK_DWN
 Text GLabel 3700 3000 0    50   Output ~ 0
-TBD
+ALT
 Text GLabel 3100 850  1    50   Input ~ 0
 Vss3.3
@@
 Wire Wire Line
 	3700 1650 3850 1650
-Text GLabel 2500 6100 0    50   Input ~ 0
+Text GLabel 2550 5000 0    50   Input ~ 0
 FX1
-Text GLabel 2500 5100 0    50   Input ~ 0
+Text GLabel 2550 5100 0    50   Input ~ 0
 FX2
-Text GLabel 2500 5000 0    50   Input ~ 0
+Text GLabel 2550 5800 0    50   Input ~ 0
 FX3
-Text GLabel 2500 4900 0    50   Input ~ 0
+Text GLabel 2550 5900 0    50   Input ~ 0
 FX4
-Text GLabel 3250 6200 2    50   Input ~ 0
+Text GLabel 2550 6000 0    50   Input ~ 0
 FX5
-Text GLabel 2400 3600 0    50   Input ~ 0
+Text GLabel 2550 6100 0    50   Input ~ 0
 PRE_A
-Text GLabel 2400 3700 0    50   Input ~ 0
+Text GLabel 2550 6200 0    50   Input ~ 0
 PRE_B
-Text GLabel 2400 3800 0    50   Input ~ 0
+Text GLabel 3300 4900 2    50   Input ~ 0
 PRE_C
-Text GLabel 2400 3900 0    50   Input ~ 0
+Text GLabel 3300 5000 2    50   Input ~ 0
 PRE_D
-Text GLabel 3300 4900 2    50   Input ~ 0
+Text GLabel 2550 4700 0    50   Input ~ 0
 BNK_UP
-Text GLabel 3300 5100 2    50   Input ~ 0
+Text GLabel 2550 4900 0    50   Input ~ 0
 BNK_DWN
-Text GLabel 2900 3750 0    50   Input ~ 0
-TBD
-Text GLabel 3650 3550 0    50   Output ~ 0
+Text GLabel 3300 5200 2    50   Input ~ 0
+ALT
+Text GLabel 3250 6300 2    50   Output ~ 0
 LOAD
-Text GLabel 3600 3650 0    50   Output ~ 0
+Text GLabel 3250 6200 2    50   Output ~ 0
 CLK
-Text GLabel 3550 3750 0    50   Output ~ 0
+Text GLabel 3250 6100 2    50   Output ~ 0
 DIN
 Text GLabel 3350 4600 2    50   Input ~ 0
@@
 Wire Wire Line
 	3350 4600 3150 4600
-Wire Wire Line
-	3300 4900 3150 4900
-Wire Wire Line
-	3300 5100 3150 5100
-Wire Wire Line
-	2500 4900 2650 4900
-Wire Wire Line
-	2500 5000 2650 5000
-Wire Wire Line
-	2500 5100 2650 5100
-Wire Wire Line
-	2500 6100 2650 6100
-Wire Wire Line
-	3150 6200 3250 6200
 Text GLabel 3350 4400 2    50   Input ~ 0
 Vss
@@
 NoConn ~ 6150 3450
 NoConn ~ 6150 3550
+Wire Wire Line
+	2550 4700 2650 4700
+Wire Wire Line
+	2550 4900 2650 4900
+Wire Wire Line
+	2550 5000 2650 5000
+Wire Wire Line
+	2550 5100 2650 5100
+Wire Wire Line
+	3150 4900 3300 4900
+Wire Wire Line
+	3300 5000 3150 5000
+Wire Wire Line
+	3300 5200 3150 5200
+Wire Wire Line
+	3150 6100 3250 6100
+Wire Wire Line
+	3150 6200 3250 6200
+Wire Wire Line
+	3150 6300 3250 6300
+Wire Wire Line
+	2650 6200 2550 6200
+Wire Wire Line
+	2650 6100 2550 6100
+Wire Wire Line
+	2650 6000 2550 6000
+Wire Wire Line
+	2650 5900 2550 5900
+Wire Wire Line
+	2650 5800 2550 5800
 $EndSCHEMATC
